File: Schematic/Kicad_Schematic/Flipper_Zero_DIY/Block_Diagram.kicad_sch (KiCad schematic)
At the start: 6 parts

Commit message: finished peripherals
Parts:
- Buttons1, CC1, LCD1, Periphery1, Power1: now left out of the parts list
Connections:
- net at CC1. (SPI_R_SCK), MCU1. (iBTN): now also Periphery1. (iBTN)
- net at MCU1. (iBTN): now also Power1. (PERIPH_POWER); no longer CC1. (SPI_R_SCK)
- net at Buttons1. (RESET), MCU1. (iBTN): now also Power1. (PERIPH_POWER)
- net at LCD1. (SPI_D_SCK): now also Periphery1. (iBTN); no longer MCU1. (iBTN)
- new net: CC1. (SPI_R_SCK), MCU1. (iBTN) (x3)
- new net: CC1. (SPI_R_SCK), MCU1. (iBTN), Periphery1. (iBTN) (x2)
- new net: Buttons1. (RESET), MCU1. (iBTN) (x5)
- new net: Buttons1. (RESET), MCU1. (iBTN), Periphery1. (iBTN)
- new net: LCD1. (SPI_D_SCK), MCU1. (iBTN) (x2)
- new net: LCD1. (SPI_D_SCK), MCU1. (iBTN), Periphery1. (iBTN) (x2)
- new net: MCU1. (iBTN), Periphery1. (iBTN) (x25)
- new net: MCU1. (iBTN), Periphery1. (iBTN), Power1. (PERIPH_POWER) (x2)
Changed lines of the file:
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@@
   )
   (symbol (lib_id "Flipper_Zero_Lib:Flipper_Zero_CC101_Block") (at 196.85 97.79 0) (unit 1)
-    (in_bom yes) (on_board yes) (dnp no) (fields_autoplaced)
+    (in_bom no) (on_board no) (dnp no) (fields_autoplaced)
     (property "Reference" "CC1" (at 224.79 90.9292 0)
       (effects (font (size 1.27 1.27)) (justify left))
@@
       (effects (font (size 1.27 1.27)) hide)
     )
+    (property "Sim.Enable" "0" (at 196.85 97.79 0)
+      (effects (font (size 1.27 1.27)) hide)
+    )
     (pin "")
     (pin "")
@@
       (effects (font (size 1.27 1.27)) hide)
     )
+    (property "Sim.Enable" "0" (at 146.685 96.52 0)
+      (effects (font (size 1.27 1.27)) hide)
+    )
     (pin "")
     (pin "")
@@
   )
   (symbol (lib_id "Flipper_Zero_Lib:Flipper_Zero_Button_Block") (at 146.685 163.83 0) (unit 1)
-    (in_bom yes) (on_board yes) (dnp no) (fields_autoplaced)
+    (in_bom no) (on_board no) (dnp no) (fields_autoplaced)
     (property "Reference" "Buttons1" (at 163.195 172.5958 0)
       (effects (font (size 1.27 1.27)) (justify left))
@@
       (effects (font (size 1.27 1.27)) hide)
     )
+    (property "Sim.Enable" "0" (at 146.685 163.83 0)
+      (effects (font (size 1.27 1.27)) hide)
+    )
     (pin "")
     (pin "")
@@
   )
   (symbol (lib_id "Flipper_Zero_Lib:Flipper_Zero_LCD_BLOCK") (at 194.31 44.45 0) (unit 1)
-    (in_bom yes) (on_board yes) (dnp no) (fields_autoplaced)
+    (in_bom no) (on_board no) (dnp no) (fields_autoplaced)
     (property "Reference" "LCD1" (at 220.98 48.3842 0)
       (effects (font (size 1.27 1.27)) (justify left))
@@
       (effects (font (size 1.27 1.27)) hide)
     )
+    (property "Sim.Enable" "0" (at 194.31 44.45 0)
+      (effects (font (size 1.27 1.27)) hide)
+    )
     (pin "")
     (pin "")
@@
   )
   (symbol (lib_id "Flipper_Zero_Lib:Flipper_Zero_Periphery_Block") (at 78.105 78.74 0) (unit 1)
-    (in_bom yes) (on_board yes) (dnp no) (fields_autoplaced)
+    (in_bom no) (on_board no) (dnp no) (fields_autoplaced)
     (property "Reference" "Periphery1" (at 74.295 39.37 0)
       (effects (font (size 1.27 1.27)))
@@
       (effects (font (size 1.27 1.27)) hide)
     )
+    (property "Sim.Enable" "0" (at 78.105 78.74 0)
+      (effects (font (size 1.27 1.27)) hide)
+    )
     (pin "")
     (pin "")
@@
   )
   (symbol (lib_id "Flipper_Zero_Lib:Flipper_Zero_Power_Block") (at 196.215 121.92 0) (unit 1)
-    (in_bom yes) (on_board yes) (dnp no) (fields_autoplaced)
+    (in_bom no) (on_board no) (dnp no) (fields_autoplaced)
     (property "Reference" "Power1" (at 224.79 124.4666 0)
       (effects (font (size 1.27 1.27)) (justify left))
@@
       (effects (font (size 1.27 1.27)) hide)
     )
+    (property "Sim.Enable" "0" (at 196.215 121.92 0)
+      (effects (font (size 1.27 1.27)) hide)
+    )
