File: Schematic/Kicad_Schematic/Flipper_Zero_DIY/Buttons.kicad_sch (KiCad schematic)
At the start: 0 parts

Commit message: finished Su-1-GHz-CC1101
Other:
- company: Flipper Devices Inc. -> Originally from : Flipper Devices Inc.
Changed lines of the file:
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@@
     (title "Flipper Device DIY")
     (rev "13.F7B9C6")
-    (company "Flipper Devices Inc.")
+    (company "Originally from : Flipper Devices Inc.")
+    (comment 1 "DIY Version 1.0")
   )
 )

Commit message: Finished the button Schematic and so the main PCB Schematic :)
Parts:
- added C85: 100nF, Capacitor_SMD:C_0402_1005Metric, symbol Device:C
- added C86, C87: 10uF, Capacitor_SMD:C_0402_1005Metric, symbol Device:C
- added DD8: NC7SZ125M5X, Package_TO_SOT_SMD:SOT-23-5, symbol 74xGxx:NC7SZ125M5X
- added R49, R50, R51, R53, R61, R62: 10k, Resistor_SMD:R_0402_1005Metric, symbol Device:R
- added R52: DNP, Resistor_SMD:R_0402_1005Metric, symbol Device:R
- added R54, R55, R56, R57, R58, R59: 330, Resistor_SMD:R_0402_1005Metric, symbol Device:R
- added R60, R64: 100k, Resistor_SMD:R_0402_1005Metric, symbol Device:R
- added R63: 510, Resistor_SMD:R_0402_1005Metric, symbol Device:R
- added SW3, SW4, SW5, SW6, SW7, SW8: SKRMAAE010, footprints:SKRMAAE010_AAL, symbol Switch:SW_Push
- added VD27, VD29, VD30, VD33, VD34, VD35: ESD241B1W0201E6327XTSA1, Diode_SMD:D_0201_0603Metric, symbol Diode:SZESD9B5.0ST5G
- added VD28, VD31, VD32: 1N4148X, Diode_SMD:D_SOD-523, symbol Device:D
Connections:
- new net: R49.1, R59.2, SW8.1, VD34.1 (A1)
- new net: R52.1, R54.2, R60.2, SW3.1, VD27.1 (A1), VD28.2 (A)
- new net: R51.1, R56.2, SW5.1, VD29.1 (A1)
- new net: R55.2, R61.2, SW4.1, VD35.1 (A1)
- new net: C86.1, DD8.1 (IN1), R60.1, VD28.1 (K)
- new net: R50.1, R58.2, SW7.1, VD33.1 (A1)
- new net: R53.1, R57.2, R64.2, SW6.1, VD30.1 (A1), VD31.2 (A)
- new net: C87.1, DD8.2 (IN2), R64.1, VD31.1 (K)
- new net: R63.2, VD32.2 (A)
- new net: DD8.4 (OUT), VD32.1 (K)
- new net +3V3: C85.1, DD8.5 (VCC), R49.2, R50.2, R51.2, R52.2, R53.2, R62.2, SW4.2
- new net BUTTON_BACK: R54.1
- new net BUTTON_DOWN: R59.1
- new net BUTTON_LEFT: R57.1
- new net BUTTON_OK: R55.1
- new net BUTTON_RIGHT: R56.1
- new net BUTTON_UP: R58.1
- new net GNDREF: C85.2, C86.2, C87.2, DD8.3 (GND), R61.1, SW3.2, SW5.2, SW6.2, SW7.2, SW8.2, VD27.2 (A2), VD29.2 (A2), VD30.2 (A2), VD33.2 (A2), VD34.2 (A2), VD35.2 (A2)
- new net RESET: R62.1, R63.1
