File: Schematic/Kicad_Schematic/Flipper_Zero_DIY/LCD-display.kicad_sch (KiCad schematic)
At the start: 0 parts

Commit message: Finished LCD-Display Schematic
Parts:
- added C48: 10uF, Capacitor_SMD:C_0603_1608Metric, symbol Device:C
- added C49: 100nF, Capacitor_SMD:C_0402_1005Metric, symbol Device:C
- added C50, C51, C52, C53, C55, C56, C57, C58: DNP, Capacitor_SMD:C_0402_1005Metric, symbol Device:C
- added C54: 2.2uF, Capacitor_SMD:C_0402_1005Metric, symbol Device:C
- added R17, R18: DNP, Resistor_SMD:R_0402_1005Metric, symbol Device:R
- added X5: FH34SRJ-30S-0.5SH(50), footprints:CONN30x1_FH34SRJ-30S-0.5SH50_HIR, symbol Connector2:Conn_01x32_Female
Connections:
- new net: C51.1, X5.18 (Pin_18)
- new net: C51.2, C54.1, X5.19 (Pin_19)
- new net: C56.2, X5.25 (Pin_25)
- new net: C50.1, X5.17 (Pin_17)
- new net: C52.2, X5.23 (Pin_23)
- new net: C58.2, X5.27 (Pin_27)
- new net: C54.2, X5.20 (Pin_20)
- new net: C53.1, X5.21 (Pin_21)
- new net: C53.2, X5.22 (Pin_22)
- new net: C55.2, X5.24 (Pin_24)
- new net: C57.2, X5.26 (Pin_26)
- new net +3V3: C48.1, C49.1, X5.10 (Pin_10), X5.11 (Pin_11), X5.12 (Pin_12), X5.15 (Pin_15), X5.5 (Pin_5), X5.6 (Pin_6), X5.7 (Pin_7), X5.8 (Pin_8), X5.9 (Pin_9)
- new net DISPLAY_CS: R17.2, X5.2 (Pin_2)
- new net DISPLAY_DI: X5.4 (Pin_4)
- new net DISPLAY_RST: R18.2, X5.3 (Pin_3)
- new net GNDREF: C48.2, C49.2, C50.2, C52.1, C55.1, C56.1, C57.1, C58.1, R17.1, R18.1, X5.16 (Pin_16), X5.28 (Pin_28), X5.29 (Pin_29), X5.31 (Pin_31), X5.32 (Pin_32)
- new net SPI_D_MOSI: X5.14 (Pin_14)
- new net SPI_D_SCK: X5.13 (Pin_13)
Other:
- note added: "C86"
- note added: "CAP1+"
- note added: "CAP1-"
- note added: "CAP2+"
- note added: "CAP2-"
- note added: "CAP3+"
- note added: "GND"
- note added: "LCD_CS"
- note added: "LCD_D/I"
- note added: "LCD_DB0"
- note added: "LCD_DB1"
- note added: "LCD_DB2"
- note added: "LCD_DB3"
- note added: "LCD_DB4"
- note added: "LCD_DB5"
- note added: "LCD_DB6(CLK)"
- note added: "LCD_DB7(Data)"
- note added: "LCD_R/W"
- note added: "LCD_RD(E)"
- note added: "LCD_RESET"
- note added: "PS"
- note added: "V0"
- note added: "V1"
- note added: "V2"
- note added: "V3"
- note added: "V4"
- note added: "Vdd"
- note added: "Vout"
- note added: "shell"

Commit message: finished Su-1-GHz-CC1101
Parts:
- added HG3: ERC12864FAMF03-1-S7, Connector_PinHeader_2.00mm:PinHeader_1x02_P2.00mm_Vertical_SMD_Pin1Left, symbol Connector:Conn_01x02_Socket
- added R19: 0, Resistor_SMD:R_0402_1005Metric, symbol Device:R
Connections:
- new net: HG3.1 (Pin_1), R19.2
- new net LCD_LED: HG3.2 (Pin_2)
- new net SYS: R19.1
Other:
- note added: "Its not a special LCD -_-"
- note added: "https://www.buydisplay.com/download/manual/ERC12864-4.10-S7_Series_Datasheet.pdf"
- company: Flipper Devices Inc. -> Originally from : Flipper Devices Inc.
- moved on the sheet: C48, C49, C50, C51, C52, C53, C54, C55, C56, C57, C58, R17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

Commit message: added all changes to the changelog
Other:
- note added: "LCD Data Connector"
- note added: "LCD Power Connector"
Changed lines of the file:
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@@
+    (stroke (width 0) (type default))
+  )
+  (polyline (pts (xy 60.325 36.83) (xy 13.335 36.83))
     (stroke (width 0) (type default))
   )
@@
     (stroke (width 0) (type default))
   )
+  (polyline (pts (xy 13.335 130.81) (xy 13.97 130.81))
+    (stroke (width 0) (type default))
+  )
   (wire (pts (xy 57.785 93.98) (xy 57.785 92.075))
     (stroke (width 0) (type default))
@@
     (stroke (width 0) (type default))
   )
+  (polyline (pts (xy 60.325 12.7) (xy 60.325 36.83))
+    (stroke (width 0) (type default))
+  )
   (wire (pts (xy 41.275 104.775) (xy 41.275 102.87))
     (stroke (width 0) (type default))
@@
     (stroke (width 0) (type default))
   )
+  (polyline (pts (xy 124.46 130.81) (xy 124.46 114.3))
+    (stroke (width 0) (type default))
+  )
   (wire (pts (xy 40.64 68.58) (xy 113.665 68.58))
     (stroke (width 0) (type default))
@@
     (stroke (width 0) (type default))
   )
+  (polyline (pts (xy 13.335 36.83) (xy 13.335 130.81))
+    (stroke (width 0) (type default))
+  )
   (wire (pts (xy 109.22 45.72) (xy 109.22 48.26))
     (stroke (width 0) (type default))
@@
     (stroke (width 0) (type default))
   )
+  (polyline (pts (xy 13.97 130.81) (xy 124.46 130.81))
+    (stroke (width 0) (type default))
+  )
   (wire (pts (xy 87.63 90.805) (xy 81.28 90.805))
     (stroke (width 0) (type default))
   )
+  (polyline (pts (xy 124.46 114.3) (xy 146.05 114.3))
+    (stroke (width 0) (type default))
+  )
   (wire (pts (xy 86.995 63.5) (xy 113.665 63.5))
     (stroke (width 0) (type default))
@@
     (stroke (width 0) (type default))
   )
+  (polyline (pts (xy 146.05 12.7) (xy 60.325 12.7))
+    (stroke (width 0) (type default))
+  )
   (wire (pts (xy 52.705 78.74) (xy 52.705 104.775))
     (stroke (width 0) (type default))
@@
     (stroke (width 0) (type default))
   )
+  (polyline (pts (xy 146.05 114.3) (xy 146.05 12.7))
+    (stroke (width 0) (type default))
+  )
   (wire (pts (xy 96.52 118.745) (xy 96.52 96.52))
     (stroke (width 0) (type default))
   )
+  (rectangle (start 150.495 28.575) (end 197.485 83.82)
+    (stroke (width 0) (type default))
+    (fill (type none))
+  )
   (text "LCD_DB2" (at 119.38 51.435 0)
     (effects (font (size 1.27 1.27)) (justify left bottom))
@@
     (effects (font (size 1.27 1.27)) (justify left bottom))
   )
+  (text "LCD Data\nConnector" (at 26.035 53.34 0)
+    (effects (font (size 4 4) bold) (justify left bottom))
+  )
   (text "Vdd" (at 119.38 66.675 0)
     (effects (font (size 1.27 1.27)) (justify left bottom))
@@
     (effects (font (size 1.27 1.27)) (justify left bottom))
   )
+  (text "LCD Power\nConnector" (at 151.13 41.91 0)
+    (effects (font (size 4 4) bold) (justify left bottom))
+  )
   (text "CAP1-" (at 119.38 76.835 0)
