File: Schematic/Kicad_Schematic/Flipper_Zero_DIY/MCU-STM32WB55.kicad_sch (KiCad schematic)
At the start: 61 parts, among them X1 105450-0101

Commit message: finished Su-1-GHz-CC1101
Parts:
- DD1: footprint footprints:STM32WB55RGV6TR -> Package_DFN_QFN:QFN-20-1EP_4x4mm_P0.5mm_EP2.5x2.5mm
Other:
- company: Flipper Devices Inc. -> Originally from : Flipper Devices Inc.
Changed lines of the file:
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@@
     (title "Flipper Device DIY")
     (rev "13.F7B9C6")
-    (company "Flipper Devices Inc.")
+    (company "Originally from : Flipper Devices Inc.")
+    (comment 1 "DIY Version 1.0")
   )
   (junction (at 200.025 69.215) (diameter 0) (color 0 0 0 0)
@@
       (effects (font (size 1.27 1.27)))
     )
-    (property "Footprint" "footprints:STM32WB55RGV6TR" (at 143.51 61.595 0)
-      (effects (font (size 1.27 1.27)) hide)
-    )
+    (property "Footprint" "Package_DFN_QFN:QFN-20-1EP_4x4mm_P0.5mm_EP2.5x2.5mm" (at 143.51 61.595 0)
+      (effects (font (size 1.27 1.27)) hide)
+    )

Commit message: Finished the button Schematic and so the main PCB Schematic :)
Parts:
- ANT1: footprint footprints:ANT_1001312_AVX -> footprints:SKRMAAE010_AAL
- VD1, VD2, VD26, VD3: footprint Diode_SMD:D_SOD-923 -> Diode_SMD:D_0201_0603Metric
Changed lines of the file:
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@@
       (effects (font (size 1.27 1.27)) (justify right))
     )
-    (property "Footprint" "Diode_SMD:D_SOD-923" (at 66.04 93.345 0)
+    (property "Footprint" "Diode_SMD:D_0201_0603Metric" (at 66.04 93.345 0)
       (effects (font (size 1.27 1.27)) hide)
     )
@@
       (effects (font (size 1.27 1.27)) (justify left))
     )
-    (property "Footprint" "footprints:ANT_1001312_AVX" (at 264.795 97.79 0)
+    (property "Footprint" "footprints:SKRMAAE010_AAL" (at 264.795 97.79 0)
       (effects (font (size 1.27 1.27)) hide)
     )
@@
       (effects (font (size 1.27 1.27)) (justify right))
     )
-    (property "Footprint" "Diode_SMD:D_SOD-923" (at 57.15 33.02 0)
+    (property "Footprint" "Diode_SMD:D_0201_0603Metric" (at 57.15 33.02 0)
       (effects (font (size 1.27 1.27)) hide)
     )
@@
       (effects (font (size 1.27 1.27)) (justify right))
     )
-    (property "Footprint" "Diode_SMD:D_SOD-923" (at 73.66 93.345 0)
+    (property "Footprint" "Diode_SMD:D_0201_0603Metric" (at 73.66 93.345 0)
       (effects (font (size 1.27 1.27)) hide)
     )
@@
       (effects (font (size 1.27 1.27)) (justify right))
     )
-    (property "Footprint" "Diode_SMD:D_SOD-923" (at 233.045 136.525 0)
-      (effects (font (size 1.27 1.27)) hide)
-    )
+    (property "Footprint" "Diode_SMD:D_0201_0603Metric" (at 233.045 136.525 0)
+      (effects (font (size 1.27 1.27)) hide)
+    )

Commit message: eddited some footprints
Parts:
- ANT1: footprint footprints:SKRMAAE010_AAL -> footprints:ANT_1001312_AVX
Changed lines of the file:
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@@
       (effects (font (size 1.27 1.27)) (justify left))
     )
-    (property "Footprint" "footprints:SKRMAAE010_AAL" (at 264.795 97.79 0)
+    (property "Footprint" "footprints:ANT_1001312_AVX" (at 264.795 97.79 0)
       (effects (font (size 1.27 1.27)) hide)
     )

Commit message: added all changes to the changelog
Changed lines of the file:
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@@
     (stroke (width 0) (type default))
   )
-  (wire (pts (xy 185.42 175.26) (xy 191.77 175.26))
+  (wire (pts (xy 185.42 175.26) (xy 193.04 175.26))
     (stroke (width 0) (type default))
   )
@@
     (stroke (width 0) (type default))
   )
-  (wire (pts (xy 215.9 74.295) (xy 215.9 79.375))
+  (wire (pts (xy 215.9 83.82) (xy 215.9 79.375))
     (stroke (width 0) (type default))
   )
@@
     (stroke (width 0) (type default))
   )
-  (wire (pts (xy 220.98 74.295) (xy 215.9 74.295))
+  (wire (pts (xy 221.615 83.82) (xy 215.9 83.82))
     (stroke (width 0) (type default))
   )
@@
   (symbol (lib_id "power:+3V3") (at 91.44 62.865 0) (unit 1)
     (in_bom yes) (on_board yes) (dnp no)
-    (property "Reference" "#PWR010" (at 91.44 66.675 0)
+    (property "Reference" "#PWR055" (at 91.44 66.675 0)
       (effects (font (size 1.27 1.27)) hide)
     )
@@
     (instances
       (project "Flipper_Zero_DIY"
-        (path "/6fd3b1c7-f4ee-4f40-ae71-a0439f037db8/574ce9ea-c3fa-46b8-8d0b-f8692bcd0c57"
-          (reference "#PWR010") (unit 1)
-        )
         (path "/6fd3b1c7-f4ee-4f40-ae71-a0439f037db8/3c4a817d-5c25-43ae-9205-7ae290fb93d7"
           (reference "#PWR055") (unit 1)
@@
     )
   )
-  (symbol (lib_id "power:+3V3") (at 191.77 175.26 270) (unit 1)
-    (in_bom yes) (on_board yes) (dnp no)
-    (property "Reference" "#PWR077" (at 187.96 175.26 0)
-      (effects (font (size 1.27 1.27)) hide)
-    )
-    (property "Value" "+3V3" (at 191.77 177.165 90)
-      (effects (font (size 1.27 1.27)) (justify left))
-    )
-    (property "Footprint" "" (at 191.77 175.26 0)
-      (effects (font (size 1.27 1.27)) hide)
-    )
-    (property "Datasheet" "" (at 191.77 175.26 0)
+  (symbol (lib_id "power:+3V3") (at 193.04 175.26 270) (unit 1)
+    (in_bom yes) (on_board yes) (dnp no)
+    (property "Reference" "#PWR077" (at 189.23 175.26 0)
+      (effects (font (size 1.27 1.27)) hide)
+    )
+    (property "Value" "+3V3" (at 193.04 177.165 90)
+      (effects (font (size 1.27 1.27)) (justify left))
+    )
+    (property "Footprint" "" (at 193.04 175.26 0)
+      (effects (font (size 1.27 1.27)) hide)
+    )
+    (property "Datasheet" "" (at 193.04 175.26 0)
       (effects (font (size 1.27 1.27)) hide)
     )
@@
     )
   )
-  (symbol (lib_id "Connector:TestPoint") (at 220.98 74.295 270) (unit 1)
-    (in_bom yes) (on_board yes) (dnp no)
-    (property "Reference" "TP49" (at 224.282 80.01 90)
-      (effects (font (size 1.27 1.27)) hide)
-    )
-    (property "Value" "D_SCK" (at 225.425 74.295 90)
-      (effects (font (size 1.27 1.27)) (justify left))
-    )
-    (property "Footprint" "TestPoint:TestPoint_Pad_1.0x1.0mm" (at 220.98 79.375 0)
-      (effects (font (size 1.27 1.27)) hide)
-    )
-    (property "Datasheet" "~" (at 220.98 79.375 0)
-      (effects (font (size 1.27 1.27)) hide)
-    )
+  (symbol (lib_id "Connector:TestPoint") (at 221.615 83.82 270) (unit 1)
+    (in_bom yes) (on_board yes) (dnp no)
+    (property "Reference" "TP49" (at 224.917 89.535 90)
+      (effects (font (size 1.27 1.27)) hide)
+    )
+    (property "Value" "D_SCK" (at 226.06 83.82 90)
+      (effects (font (size 1.27 1.27)) (justify left))
+    )
+    (property "Footprint" "TestPoint:TestPoint_Pad_1.0x1.0mm" (at 221.615 88.9 0)
+      (effects (font (size 1.27 1.27)) hide)
+    )
+    (property "Datasheet" "~" (at 221.615 88.9 0)
+      (effects (font (size 1.27 1.27)) hide)
+    )
