File: Schematic/Kicad_Schematic/Flipper_Zero_DIY/Main_Block_Diagram.kicad_sch (KiCad schematic)
At the start: 6 parts

Commit message: finished Su-1-GHz-CC1101
Connections:
- net at CC1. (SPI_R_SCK), MCU1. (iBTN): now also Periphery1. (iBTN)
- net at MCU1. (iBTN): now also Power1. (PERIPH_POWER); no longer CC1. (SPI_R_SCK)
- net at Buttons1. (RESET), MCU1. (iBTN): now also Power1. (PERIPH_POWER)
- net at LCD1. (SPI_D_SCK): now also Periphery1. (iBTN); no longer MCU1. (iBTN)
- new net: CC1. (SPI_R_SCK), MCU1. (iBTN) (x3)
- new net: CC1. (SPI_R_SCK), MCU1. (iBTN), Periphery1. (iBTN) (x2)
- new net: Buttons1. (RESET), MCU1. (iBTN) (x5)
- new net: Buttons1. (RESET), MCU1. (iBTN), Periphery1. (iBTN)
- new net: LCD1. (SPI_D_SCK), MCU1. (iBTN) (x2)
- new net: LCD1. (SPI_D_SCK), MCU1. (iBTN), Periphery1. (iBTN) (x2)
- new net: MCU1. (iBTN), Periphery1. (iBTN) (x25)
- new net: MCU1. (iBTN), Periphery1. (iBTN), Power1. (PERIPH_POWER) (x2)
Other:
- company: Flipper Devices Inc. -> Originally from : Flipper Devices Inc.
Changed lines of the file:
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@@
     (title "Flipper Device DIY")
     (rev "13.F7B9C6")
-    (company "Flipper Devices Inc.")
+    (company "Originally from : Flipper Devices Inc.")
+    (comment 1 "DIY Version 1.0")
   )
   (junction (at 154.305 159.385) (diameter 0) (color 0 0 0 0)

Commit message: added all changes to the changelog
Parts:
- renumbered CC1 to CC1101
Connections:
- net at CC1101. (SPI_R_SCK), MCU1. (iBTN): now also Periphery1. (iBTN)
- net at MCU1. (iBTN): now also Power1. (PERIPH_POWER); no longer CC1101. (SPI_R_SCK)
- net at Buttons1. (RESET), MCU1. (iBTN): now also Power1. (PERIPH_POWER)
- net at LCD1. (SPI_D_SCK): now also Periphery1. (iBTN); no longer MCU1. (iBTN)
- new net: CC1101. (SPI_R_SCK), MCU1. (iBTN) (x3)
- new net: CC1101. (SPI_R_SCK), MCU1. (iBTN), Periphery1. (iBTN) (x2)
- new net: Buttons1. (RESET), MCU1. (iBTN) (x5)
- new net: Buttons1. (RESET), MCU1. (iBTN), Periphery1. (iBTN)
- new net: LCD1. (SPI_D_SCK), MCU1. (iBTN) (x2)
- new net: LCD1. (SPI_D_SCK), MCU1. (iBTN), Periphery1. (iBTN) (x2)
- new net: MCU1. (iBTN), Periphery1. (iBTN) (x25)
- new net: MCU1. (iBTN), Periphery1. (iBTN), Power1. (PERIPH_POWER) (x2)
Changed lines of the file:
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@@
   (symbol (lib_id "Flipper_Zero_Lib:Flipper_Zero_CC101_Block") (at 196.85 97.79 0) (unit 1)
     (in_bom no) (on_board no) (dnp no) (fields_autoplaced)
-    (property "Reference" "CC1" (at 224.79 90.9292 0)
+    (property "Reference" "CC1101" (at 224.79 90.9292 0)
       (effects (font (size 1.27 1.27)) (justify left))
     )
@@
     (instances
       (project "Flipper_Zero_DIY"
-        (path "/6fd3b1c7-f4ee-4f40-ae71-a0439f037db8"
-          (reference "CC1") (unit 1)
-        )
         (path "/6fd3b1c7-f4ee-4f40-ae71-a0439f037db8/8de03230-0fbb-4dc8-83dd-160a4cc10118"
           (reference "CC1101") (unit 1)
@@
     (instances
       (project "Flipper_Zero_DIY"
-        (path "/6fd3b1c7-f4ee-4f40-ae71-a0439f037db8"
+        (path "/6fd3b1c7-f4ee-4f40-ae71-a0439f037db8/8de03230-0fbb-4dc8-83dd-160a4cc10118"
           (reference "MCU1") (unit 1)
         )
-        (path "/6fd3b1c7-f4ee-4f40-ae71-a0439f037db8/8de03230-0fbb-4dc8-83dd-160a4cc10118"
-          (reference "MCU1") (unit 1)
-        )
       )
     )
@@
     (instances
       (project "Flipper_Zero_DIY"
-        (path "/6fd3b1c7-f4ee-4f40-ae71-a0439f037db8"
+        (path "/6fd3b1c7-f4ee-4f40-ae71-a0439f037db8/8de03230-0fbb-4dc8-83dd-160a4cc10118"
           (reference "Buttons1") (unit 1)
         )
-        (path "/6fd3b1c7-f4ee-4f40-ae71-a0439f037db8/8de03230-0fbb-4dc8-83dd-160a4cc10118"
-          (reference "Buttons1") (unit 1)
-        )
       )
     )
@@
     (instances
       (project "Flipper_Zero_DIY"
-        (path "/6fd3b1c7-f4ee-4f40-ae71-a0439f037db8"
+        (path "/6fd3b1c7-f4ee-4f40-ae71-a0439f037db8/8de03230-0fbb-4dc8-83dd-160a4cc10118"
           (reference "LCD1") (unit 1)
         )
-        (path "/6fd3b1c7-f4ee-4f40-ae71-a0439f037db8/8de03230-0fbb-4dc8-83dd-160a4cc10118"
-          (reference "LCD1") (unit 1)
-        )
       )
     )
@@
     (instances
       (project "Flipper_Zero_DIY"
-        (path "/6fd3b1c7-f4ee-4f40-ae71-a0439f037db8"
+        (path "/6fd3b1c7-f4ee-4f40-ae71-a0439f037db8/8de03230-0fbb-4dc8-83dd-160a4cc10118"
           (reference "Periphery1") (unit 1)
         )
-        (path "/6fd3b1c7-f4ee-4f40-ae71-a0439f037db8/8de03230-0fbb-4dc8-83dd-160a4cc10118"
-          (reference "Periphery1") (unit 1)
-        )
       )
     )
@@
     (instances
       (project "Flipper_Zero_DIY"
-        (path "/6fd3b1c7-f4ee-4f40-ae71-a0439f037db8"
+        (path "/6fd3b1c7-f4ee-4f40-ae71-a0439f037db8/8de03230-0fbb-4dc8-83dd-160a4cc10118"
           (reference "Power1") (unit 1)
-        )
-        (path "/6fd3b1c7-f4ee-4f40-ae71-a0439f037db8/8de03230-0fbb-4dc8-83dd-160a4cc10118"
-          (reference "Power1") (unit 1)

Commit message: ported project to KiCad 8.0 and ploted current (NOT FINISHED) diy schematics
Connections:
- net at CC1101. (SPI_R_SCK), MCU1. (iBTN): now also Periphery1. (iBTN)
- net at MCU1. (iBTN): now also Power1. (PERIPH_POWER); no longer CC1101. (SPI_R_SCK)
- net at Buttons1. (RESET), MCU1. (iBTN): now also Power1. (PERIPH_POWER)
- net at LCD1. (SPI_D_SCK): now also Periphery1. (iBTN); no longer MCU1. (iBTN)
- new net: CC1101. (SPI_R_SCK), MCU1. (iBTN) (x3)
- new net: CC1101. (SPI_R_SCK), MCU1. (iBTN), Periphery1. (iBTN) (x2)
- new net: Buttons1. (RESET), MCU1. (iBTN) (x5)
- new net: Buttons1. (RESET), MCU1. (iBTN), Periphery1. (iBTN)
- new net: LCD1. (SPI_D_SCK), MCU1. (iBTN) (x2)
- new net: LCD1. (SPI_D_SCK), MCU1. (iBTN), Periphery1. (iBTN) (x2)
- new net: MCU1. (iBTN), Periphery1. (iBTN) (x25)
- new net: MCU1. (iBTN), Periphery1. (iBTN), Power1. (PERIPH_POWER) (x2)
