File: Schematic/Kicad_Schematic/Flipper_Zero_DIY/NFC.kicad_sch (KiCad schematic)
At the start: 0 parts

Commit message: finished Su-1-GHz-CC1101
Other:
- company: Flipper Devices Inc. -> Originally from : Flipper Devices Inc.
Changed lines of the file:
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@@
     (title "Flipper Device DIY")
     (rev "13.F7B9C6")
-    (company "Flipper Devices Inc.")
+    (company "Originally from : Flipper Devices Inc.")
+    (comment 1 "DIY Version 1.0")
   )
 )

Commit message: finished NFC_RFID-Blockdia and NFC Schematic
Parts:
- added RC1, RC10, RC3, RC8: 100pF, symbol Device:C
- added RC11, RC15: 6pF, symbol Device:C
- added RC12, RC13, RC14, RC22, RC23, RC47, RC48: DNP, symbol Device:C
- added RC16, RC18, RC20, RC24, RC26, RC28, RC30, RC32: 10nF, symbol Device:C
- added RC17, RC19, RC21, RC25, RC27, RC29, RC31, RC33: 2.2uF, symbol Device:C
- added RC2, RC9: 10pF, symbol Device:C
- added RC4, RC6: 680pF, symbol Device:C
- added RC5, RC7: 62pF, symbol Device:C
- added RDD1: ST25R3916-AQWT, VFQFPN32_5X5_WETTABLE_STM, symbol ST25R3916-AQWT:ST25R3916-AQWT
- added RL1, RL2: 270nH, symbol Device:L
- added RR1, RR2: 0, symbol Device:R
- added RX6, RX7: FDX0022A1, symbol Device:Antenna
- added RZQ1: XRCGB27M120F3M00R0, symbol Device:Crystal_GND2_Small
- added TP62: RCP1, symbol Connector:TestPoint
- added TP63: RCP2, symbol Connector:TestPoint
- added TP64: RAN2, symbol Connector:TestPoint
- added TP65: RANT1, symbol Connector:TestPoint_2Pole
- added TP66: RAN1, symbol Connector:TestPoint
- added TP67: RANT2, symbol Connector:TestPoint_2Pole
- added TP68: RCP3, symbol Connector:TestPoint
Connections:
- new net: RDD1.2 (CSO), TP63.1
- new net: RC26.2, RC27.2, RDD1.11 (VDD_AM)
- new net: RDD1.13 (RFO1), RL1.1
- new net: RC3.1, RC4.2, RC47.1, RL1.2
- new net: RC30.2, RC31.2, RDD1.24 (AGDC)
- new net: RC48.1, RC6.1, RC8.1, RL2.2
- new net: RC48.2, RC7.1, RC8.2, RC9.2, RR2.1
- new net: RC11.2, RDD1.4 (XTO), RZQ1.1
- new net: RC16.2, RC17.2, RDD1.3 (VDD_D)
- new net: RDD1.15 (RFO2), RL2.1
- new net: RDD1.25 (CSI), TP62.1
- new net: RC2.2, RC3.2, RC47.2, RC5.2, RR1.1
- new net: RR2.2, RX7.1 (A), TP66.1, TP67.1
- new net: RR1.2, RX6.1 (A), TP64.1, TP65.1
- new net: RC10.1, RC9.1, RDD1.23 (RFI2)
- new net: RC22.2, RC23.2, RC28.2, RC29.2, RDD1.14 (VDD_DR), RDD1.9 (VDD_RF)
- new net: RC15.2, RDD1.5 (XTI), RZQ1.3
- new net: RDD1.17 (EXT_LM), TP68.1
- new net: RC1.1, RC2.1, RDD1.22 (RFI1)
- new net: RC18.2, RC19.2, RDD1.7 (VDD_A)
- new net +3V3: RC32.2, RC33.2, RDD1.1 (VDD_IO)
- new net +5V: RC20.2, RC21.2, RC24.2, RC25.2, RDD1.10 (VDD_TX), RDD1.8 (VDD)
- new net GNDREF: RC1.2, RC10.2, RC11.1, RC12.2, RC13.2, RC14.2, RC15.1, RC16.1, RC17.1, RC18.1, RC19.1, RC20.1, RC21.1, RC22.1, RC23.1, RC24.1, RC25.1, RC26.1, RC27.1, RC28.1, RC29.1, RC30.1, RC31.1, RC32.1, RC33.1, RC4.1, RC5.1, RC6.2, RC7.2, RDD1.12 (GND_DR), RDD1.16 (GND_DR), RDD1.20 (I2C_EN), RDD1.21 (VSS), RDD1.26 (GND_A), RDD1.33 (EPAD), RDD1.6 (GND_D), RZQ1.2, TP65.2, TP67.2
- new net NFC_CS: RDD1.29 (BSS)
- new net NFC_IRQ: RDD1.27 (IRQ)
- new net SPI_R_MISO: RC14.1, RDD1.32 (MISO/SDA)
- new net SPI_R_MOSI: RC13.1, RDD1.31 (MOSI)
- new net SPI_R_SCK: RC12.1, RDD1.30 (SCLK/SCL)
- no-connect marks 0 -> 1
