File: Schematic/Kicad_Schematic/Flipper_Zero_DIY/NFC_Block_Diagram.kicad_sch (KiCad schematic)
At the start: 0 parts

Commit message: finished Su-1-GHz-CC1101
Other:
- company: Flipper Devices Inc. -> Originally from : Flipper Devices Inc.
Changed lines of the file:
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@@
     (title "Flipper Device DIY")
     (rev "13.F7B9C6")
-    (company "Flipper Devices Inc.")
+    (company "Originally from : Flipper Devices Inc.")
+    (comment 1 "DIY Version 1.0")
   )
 )

Commit message: finished NFC_RFID-Blockdia and NFC Schematic
Parts:
- added NFC1: Flipper_zero_NFC.SchDoc, symbol Flipper_Zero_Lib:NFC_BLOCK
- added PERIPHERY2: Flipper_zero_PERIPHERY.SchDoc, symbol Flipper_Zero_Lib:PERIPHERY_BLOCK
- added RFID_iBTN1: Flipper_zero_RFID_iBTN.SchDoc, symbol Flipper_Zero_Lib:RFID_iBTN_BLOCK
Connections:
- new net: NFC1. (SPI_R_SCK), PERIPHERY2. (iBTN) (x4)
- new net: NFC1. (SPI_R_SCK), RFID_iBTN1. (iBTN)
- new net: PERIPHERY2. (iBTN), RFID_iBTN1. (iBTN) (x8)
Changed lines of the file:
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@@
 (kicad_sch (version 20230121) (generator eeschema)
-  (paper "A4")
+  (paper "A5")
   (title_block
     (title "Flipper Device DIY")
@@
     (comment 1 "DIY Version 1.0")
   )
+  (wire (pts (xy 85.09 81.28) (xy 96.52 81.28))
+    (stroke (width 0) (type default))
+  )
+  (wire (pts (xy 115.57 59.69) (xy 130.175 59.69))
+    (stroke (width 0) (type default))
+  )
+  (wire (pts (xy 85.09 49.53) (xy 96.52 49.53))
+    (stroke (width 0) (type default))
+  )
+  (wire (pts (xy 130.175 59.69) (xy 130.175 74.93))
+    (stroke (width 0) (type default))
+  )
+  (wire (pts (xy 85.09 68.58) (xy 96.52 68.58))
+    (stroke (width 0) (type default))
+  )
+  (wire (pts (xy 130.175 74.93) (xy 125.73 74.93))
+    (stroke (width 0) (type default))
+  )
+  (wire (pts (xy 85.09 57.15) (xy 96.52 57.15))
+    (stroke (width 0) (type default))
+  )
+  (wire (pts (xy 85.09 78.74) (xy 96.52 78.74))
+    (stroke (width 0) (type default))
+  )
+  (wire (pts (xy 85.09 86.36) (xy 96.52 86.36))
+    (stroke (width 0) (type default))
+  )
+  (wire (pts (xy 85.09 54.61) (xy 96.52 54.61))
+    (stroke (width 0) (type default))
+  )
+  (wire (pts (xy 85.09 66.04) (xy 96.52 66.04))
+    (stroke (width 0) (type default))
+  )
+  (wire (pts (xy 85.09 52.07) (xy 96.52 52.07))
+    (stroke (width 0) (type default))
+  )
+  (wire (pts (xy 85.09 74.93) (xy 96.52 74.93))
+    (stroke (width 0) (type default))
+  )
+  (wire (pts (xy 85.09 83.82) (xy 96.52 83.82))
+    (stroke (width 0) (type default))
+  )
+  (wire (pts (xy 85.09 72.39) (xy 96.52 72.39))
+    (stroke (width 0) (type default))
+  )
+  (symbol (lib_id "Flipper_Zero_Lib:NFC_BLOCK") (at 99.06 46.99 0) (unit 1)
+    (in_bom no) (on_board no) (dnp no) (fields_autoplaced)
+    (property "Reference" "NFC1" (at 106.045 42.545 0)
+      (effects (font (size 1.27 1.27)))
+    )
+    (property "Value" "Flipper_zero_NFC.SchDoc" (at 106.045 45.085 0)
+      (effects (font (size 1.27 1.27)))
+    )
+    (property "Footprint" "" (at 99.06 46.99 0)
+      (effects (font (size 1.27 1.27)) hide)
+    )
+    (property "Datasheet" "" (at 99.06 46.99 0)
+      (effects (font (size 1.27 1.27)) hide)
+    )
+    (pin "")
+    (pin "")
+    (pin "")
+    (pin "")
+    (pin "")
+    (instances
+      (project "Flipper_Zero_DIY"
+        (path "/6fd3b1c7-f4ee-4f40-ae71-a0439f037db8/6eb83f5a-7b16-426a-9130-a087b28e79cc"
+          (reference "NFC1") (unit 1)
+        )
+      )
+    )
+  )
+  (symbol (lib_id "Flipper_Zero_Lib:PERIPHERY_BLOCK") (at 82.55 50.8 0) (unit 1)
+    (in_bom no) (on_board no) (dnp no) (fields_autoplaced)
+    (property "Reference" "PERIPHERY2" (at 74.93 43.18 0)
+      (effects (font (size 1.27 1.27)))
+    )
+    (property "Value" "Flipper_zero_PERIPHERY.SchDoc" (at 74.93 45.72 0)
+      (effects (font (size 1.27 1.27)))
+    )
+    (property "Footprint" "" (at 82.55 43.18 0)
+      (effects (font (size 1.27 1.27)) hide)
+    )
+    (property "Datasheet" "" (at 82.55 43.18 0)
+      (effects (font (size 1.27 1.27)) hide)
+    )
+    (pin "")
+    (pin "")
+    (pin "")
+    (pin "")
+    (pin "")
+    (pin "")
+    (pin "")
+    (pin "")
+    (pin "")
+    (pin "")
+    (pin "")
+    (pin "")
+    (instances
+      (project "Flipper_Zero_DIY"
+        (path "/6fd3b1c7-f4ee-4f40-ae71-a0439f037db8/6eb83f5a-7b16-426a-9130-a087b28e79cc"
+          (reference "PERIPHERY2") (unit 1)
+        )
+      )
+    )
+  )
+  (symbol (lib_id "Flipper_Zero_Lib:RFID_iBTN_BLOCK") (at 109.22 62.23 0) (unit 1)
+    (in_bom no) (on_board no) (dnp no)
+    (property "Reference" "RFID_iBTN1" (at 111.125 90.17 0)
+      (effects (font (size 1.27 1.27)))
+    )
+    (property "Value" "Flipper_zero_RFID_iBTN.SchDoc" (at 112.395 92.075 0)
+      (effects (font (size 1.27 1.27)))
+    )
+    (property "Footprint" "" (at 109.22 62.23 0)
+      (effects (font (size 1.27 1.27)) hide)
+    )
+    (property "Datasheet" "" (at 109.22 62.23 0)
+      (effects (font (size 1.27 1.27)) hide)
+    )
+    (pin "")
+    (pin "")
+    (pin "")
+    (pin "")
+    (pin "")
+    (pin "")
+    (pin "")
+    (pin "")
+    (pin "")
+    (instances
+      (project "Flipper_Zero_DIY"
+        (path "/6fd3b1c7-f4ee-4f40-ae71-a0439f037db8/6eb83f5a-7b16-426a-9130-a087b28e79cc"
+          (reference "RFID_iBTN1") (unit 1)
+        )
+      )
+    )
+  )
 )

Commit message: ported project to KiCad 8.0 and ploted current (NOT FINISHED) diy schematics
Connections:
- net at NFC1. (SPI_R_SCK): now also RFID_iBTN1. (iBTN); no longer PERIPHERY2. (iBTN)
- net at PERIPHERY2. (iBTN): now also RFID_iBTN1. (iBTN); no longer NFC1. (SPI_R_SCK)
- new net: NFC1. (SPI_R_SCK), PERIPHERY2. (iBTN) (x4)
- new net: PERIPHERY2. (iBTN), RFID_iBTN1. (iBTN) (x7)
