File: Schematic/Kicad_Schematic/Flipper_Zero_DIY/Peripherals.kicad_sch (KiCad schematic)
At the start: 84 parts, among them J2 Micro_SD_Card_Det, X6 FH34SRJ-18S-0.5SH(50), X8 2.54-WT-1X10, X9 2.54-WT-1X8

Commit message: finished peripherals
Parts:
- removed D1, D2, D3: D, symbol Device:D
- removed R10, R10B1, R10C1, R10D1, R11, R11B1, R11C1, R11D1, R32, R32B1, R32C1, R32D1, R33, R33B1, R33C1, R33D1: 51, symbol Device:R
- added R10, R11, R32, R33: 51, Resistor_SMD:R_Array_Convex_4x0402, symbol Device:R_Network04_Split
- added VD4: LED_ABGR, LED_SMD:LED_RGB_1210, symbol Device:LED_ABGR
- C59: footprint (none) -> Capacitor_SMD:C_0402_1005Metric
- C60, C61: footprint (none) -> Capacitor_SMD:C_0603_1608Metric
- C62: footprint (none) -> Capacitor_SMD:C_1206_3216Metric
- DA4: footprint YQE0012ACAC -> footprints:LP5562TMX-NOPB
- FU4: footprint (none) -> Fuse:Fuse_0402_1005Metric
- R20, R21, R22, R23, R24, R25, R26, R27, R28, R29, R30, R31, R65, R66, R67, R68, R69: footprint (none) -> Resistor_SMD:R_0402_1005Metric
- TP24, TP25, TP26, TP27, TP28, TP29, TP30, TP31, TP32, TP33, TP34, TP35, TP36, TP37, TP38, TP39: footprint (none) -> TestPoint:TestPoint_Pad_1.0x1.0mm
- VD10, VD11, VD12, VD13, VD14, VD15, VD16, VD17, VD18, VD19, VD20, VD21, VD22, VD23, VD24, VD25, VD5, VD6, VD7, VD8, VD9: footprint (none) -> Diode_SMD:D_0201_0603Metric
- VD36: footprint (none) -> Diode_SMD:D_SOD-523
- X6: footprint (none) -> footprints:18_pin_JST
- X7: renamed from J2; value Micro_SD_Card_Det -> Micro_SD; footprint (none) -> Connector_Card:microSD_HC_Hirose_DM3AT-SF-PEJM5
- X8: footprint (none) -> Connector_PinHeader_2.00mm:PinHeader_1x10_P2.00mm_Horizontal
- X9: footprint (none) -> Connector_PinHeader_2.00mm:PinHeader_1x08_P2.00mm_Horizontal
Connections:
- net PA4: now also R33.1 (R1)
- net PA6: now also R10.1 (R1)
- net PA7: now also R10.1 (R1)
- net PB2: now also R33.1 (R1)
- net PB3: now also R33.1 (R1)
- net PC0: now also R32.1 (R1)
- net PC1: now also R32.1 (R1)
- net PC3: now also R33.1 (R1)
- net SWCLK: now also R11.1 (R1)
- net SWDIO: now also R11.1 (R1)
- net SYS: now also VD4.1 (A)
- net UART1_RX: now also R32.1 (R1)
- net UART1_TX: now also R11.1 (R1)
- net iBTN: now also R32.1 (R1)
- net at X8.2 (Pin_2): now also R11.2 (R1.2)
- net at X8.4 (Pin_4): now also R11.3 (R2.2)
- net at TP29.1, X8.5 (Pin_5): now also R11.5 (R4.2)
- net at TP28.1, X8.6 (Pin_6): now also R32.2 (R1.2)
- net at TP27.1, X8.7 (Pin_7): now also R32.3 (R2.2)
- net at TP26.1, X8.8 (Pin_8): now also R32.4 (R3.2)
- net at X8.9 (Pin_9): now also R32.5 (R4.2)
- net at X9.5 (Pin_5): now also R33.3 (R2.2)
- net at R27.2: now also VD4.3 (GK)
- net at R25.2: now also VD4.4 (RK)
- net at X9.7 (Pin_7): now also R33.5 (R4.2)
- net at X9.2 (Pin_2): now also R10.3 (R2.2)
- net at X9.3 (Pin_3): now also R10.4 (R3.2)
- net at X9.4 (Pin_4): now also R33.2 (R1.2)
- net at X9.6 (Pin_6): now also R33.4 (R3.2)
- net at R30.2: now also VD4.2 (BK)
Other:
- note added: "TODO: Apply footprint"

Commit message: finished MCU schematic & new design of front shematic
Parts:
- R65, R66, R67: now not fitted
Other:
- company: (none) -> Flipper Devices Inc.
- title: (none) -> Flipper Device DIY
Changed lines of the file:
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@@
 (kicad_sch (version 20230121) (generator eeschema)
   (paper "A3")
+  (title_block
+    (title "Flipper Device DIY")
+    (rev "13.F7B9C6")
+    (company "Flipper Devices Inc.")
+  )
   (junction (at 242.57 189.865) (diameter 0) (color 0 0 0 0)
   )
@@
   )
   (symbol (lib_id "Device:R") (at 252.095 69.215 180) (unit 1)
-    (in_bom yes) (on_board yes) (dnp no)
+    (in_bom yes) (on_board yes) (dnp yes)
     (property "Reference" "R66" (at 249.555 72.39 90)
       (effects (font (size 1.27 1.27)))
@@
   )
   (symbol (lib_id "Device:R") (at 257.175 69.215 180) (unit 1)
-    (in_bom yes) (on_board yes) (dnp no)
+    (in_bom yes) (on_board yes) (dnp yes)
     (property "Reference" "R67" (at 254.635 72.39 90)
       (effects (font (size 1.27 1.27)))
@@
   )
   (symbol (lib_id "Device:R") (at 241.935 69.215 180) (unit 1)
-    (in_bom yes) (on_board yes) (dnp no)
+    (in_bom yes) (on_board yes) (dnp yes)
     (property "Reference" "R65" (at 239.395 72.39 90)
       (effects (font (size 1.27 1.27)))

Commit message: finished Su-1-GHz-CC1101
Other:
- company: Flipper Devices Inc. -> Originally from : Flipper Devices Inc.
Changed lines of the file:
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@@
     (title "Flipper Device DIY")
     (rev "13.F7B9C6")
-    (company "Flipper Devices Inc.")
+    (company "Originally from : Flipper Devices Inc.")
+    (comment 1 "DIY Version 1.0")
   )
   (junction (at 242.57 189.865) (diameter 0) (color 0 0 0 0)

Commit message: added all changes to the changelog
Parts:
- C62: now not fitted
- FU4: value Fuse -> ERB-RD2R00X; description (none) -> Electric Fuse, Fast Blow, 2A, 32VDC, 35A (IR), Surface Mount
- VD4: value LED_ABGR -> CLMUD-FKC-CHJNPM569ABB845343; footprint LED_SMD:LED_RGB_1210 -> footprints:SMD_RGB_LED_CLMUD-FKC-CHJNPM569ABB845343
- X8: footprint Connector_PinHeader_2.00mm:PinHeader_1x10_P2.00mm_Horizontal -> Connector_PinSocket_2.54mm:PinSocket_1x10_P2.54mm_Horizontal
- X9: footprint Connector_PinHeader_2.00mm:PinHeader_1x08_P2.00mm_Horizontal -> Connector_PinSocket_2.54mm:PinSocket_1x08_P2.54mm_Horizontal
Other:
- note added: "Ext. Pins 1-8"
- note added: "Ext. Pins 9-18"
- note added: "LED-Driver"
- note added: "PCB-PCB Connector"
- note added: "SD-Card"
- note removed: "TODO: Apply footprint"
- moved on the sheet: VD4
Changed lines of the file:
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@@
     (stroke (width 0) (type default))
   )
-  (wire (pts (xy 142.875 90.17) (xy 144.78 90.17))
+  (wire (pts (xy 142.875 90.17) (xy 144.145 90.17))
     (stroke (width 0) (type default))
   )
@@
     (stroke (width 0) (type default))
   )
-  (wire (pts (xy 142.875 95.25) (xy 144.78 95.25))
+  (wire (pts (xy 142.875 95.25) (xy 144.145 95.25))
     (stroke (width 0) (type default))
   )
@@
     (stroke (width 0) (type default))
   )
-  (wire (pts (xy 142.875 85.09) (xy 144.78 85.09))
+  (wire (pts (xy 142.875 85.09) (xy 144.145 85.09))
     (stroke (width 0) (type default))
   )
@@
     (stroke (width 0) (type default))
   )
-  (wire (pts (xy 154.94 90.17) (xy 157.48 90.17))
+  (wire (pts (xy 154.305 90.17) (xy 157.48 90.17))
     (stroke (width 0) (type default))
   )
@@
     (stroke (width 0) (type default))
   )
+  (rectangle (start 180.34 49.53) (end 354.965 149.225)
+    (stroke (width 0) (type default))
+    (fill (type none))
+  )
+  (rectangle (start 19.685 163.195) (end 119.38 253.365)
+    (stroke (width 0) (type default))
+    (fill (type none))
+  )
+  (rectangle (start 64.135 48.895) (end 170.815 132.08)
+    (stroke (width 0) (type default))
+    (fill (type none))
+  )
+  (rectangle (start 287.02 158.75) (end 403.225 262.255)
+    (stroke (width 0) (type default))
+    (fill (type none))
+  )
+  (rectangle (start 138.43 163.83) (end 275.59 262.89)
+    (stroke (width 0) (type default))
+    (fill (type none))
+  )
   (text "PC0" (at 252.73 215.265 0)
     (effects (font (size 1.27 1.27)) (justify left bottom))
   )
+  (text "SD-Card" (at 306.705 61.595 0)
+    (effects (font (size 4 4) bold) (justify left bottom))
+  )
   (text "PA7" (at 102.235 200.025 0)
     (effects (font (size 1.27 1.27)) (justify left bottom))
   )
-  (text "TODO: Apply footprint" (at 323.85 80.645 0)
-    (effects (font (size 1.27 1.27)) (justify left bottom))
-  )
   (text "PC3" (at 102.235 212.725 0)
     (effects (font (size 1.27 1.27)) (justify left bottom))
@@
     (effects (font (size 1.27 1.27)) (justify left bottom))
   )
+  (text "Ext. Pins 1-8" (at 28.575 177.165 0)
+    (effects (font (size 4 4) bold) (justify left bottom))
+  )
   (text "iBTN" (at 381.635 209.55 0)
     (effects (font (size 1.27 1.27)) (justify left bottom))
@@
     (effects (font (size 1.27 1.27)) (justify left bottom))
   )
+  (text "PCB-PCB Connector" (at 288.925 166.37 0)
+    (effects (font (size 4 4) bold) (justify left bottom))
+  )
   (text "RFID_PULL" (at 381.635 201.93 0)
     (effects (font (size 1.27 1.27)) (justify left bottom))
@@
     (effects (font (size 1.27 1.27)) (justify left bottom))
   )
+  (text "LED-Driver" (at 130.175 56.515 0)
+    (effects (font (size 4 4) (thickness 0.8) bold) (justify left bottom))
+  )
   (text "SPEAKER" (at 381.635 212.09 0)
     (effects (font (size 1.27 1.27)) (justify left bottom))
+  )
+  (text "Ext. Pins 9-18" (at 149.225 176.53 0)
+    (effects (font (size 4 4) bold) (justify left bottom))
   )
   (text "IR_RX" (at 381.635 217.17 0)
@@
   )
   (symbol (lib_id "Device:C_Polarized") (at 99.695 190.5 90) (unit 1)
-    (in_bom yes) (on_board yes) (dnp no)
+    (in_bom yes) (on_board yes) (dnp yes)
     (property "Reference" "C62" (at 96.52 189.23 90)
       (effects (font (size 1.27 1.27)))
@@
     )
   )
-  (symbol (lib_id "Device:LED_ABGR") (at 149.86 90.17 0) (unit 1)
-    (in_bom yes) (on_board yes) (dnp no)
-    (property "Reference" "VD4" (at 149.86 80.645 0)
-      (effects (font (size 1.27 1.27)))
-    )
-    (property "Value" "LED_ABGR" (at 149.86 80.01 0)
-      (effects (font (size 1.27 1.27)) hide)
-    )
-    (property "Footprint" "LED_SMD:LED_RGB_1210" (at 149.86 91.44 0)
-      (effects (font (size 1.27 1.27)) hide)
-    )
-    (property "Datasheet" "~" (at 149.86 91.44 0)
+  (symbol (lib_id "Device:LED_ABGR") (at 149.225 90.17 0) (unit 1)
+    (in_bom yes) (on_board yes) (dnp no)
+    (property "Reference" "VD4" (at 149.225 80.645 0)
+      (effects (font (size 1.27 1.27)))
+    )
+    (property "Value" "CLMUD-FKC-CHJNPM569ABB845343" (at 149.225 78.74 0)
+      (effects (font (size 1.27 1.27)))
+    )
+    (property "Footprint" "footprints:SMD_RGB_LED_CLMUD-FKC-CHJNPM569ABB845343" (at 149.225 91.44 0)
+      (effects (font (size 1.27 1.27)) hide)
+    )
+    (property "Datasheet" "https://www.mouser.de/datasheet/2/723/HB_CLMUD_FKC-3043388.pdf" (at 149.225 91.44 0)
       (effects (font (size 1.27 1.27)) hide)
     )
@@
       (effects (font (size 1.27 1.27)) (justify left))
     )
-    (property "Footprint" "Connector_PinHeader_2.00mm:PinHeader_1x10_P2.00mm_Horizontal" (at 252.095 207.01 0)
+    (property "Footprint" "Connector_PinSocket_2.54mm:PinSocket_1x10_P2.54mm_Horizontal" (at 252.095 207.01 0)
       (effects (font (size 1.27 1.27)) hide)
     )
@@
   (symbol (lib_id "power:+3V3") (at 367.665 167.64 0) (unit 1)
     (in_bom yes) (on_board yes) (dnp no)
-    (property "Reference" "#PWR010" (at 367.665 171.45 0)
+    (property "Reference" "#PWR048" (at 367.665 171.45 0)
       (effects (font (size 1.27 1.27)) hide)
     )
@@
     (instances
       (project "Flipper_Zero_DIY"
-        (path "/6fd3b1c7-f4ee-4f40-ae71-a0439f037db8/574ce9ea-c3fa-46b8-8d0b-f8692bcd0c57"
-          (reference "#PWR010") (unit 1)
-        )
         (path "/6fd3b1c7-f4ee-4f40-ae71-a0439f037db8/df3e630c-89cc-4e6d-867b-b681a42511f6"
           (reference "#PWR048") (unit 1)
@@
       (effects (font (size 1.27 1.27)) (justify left))
     )
-    (property "Value" "Fuse" (at 92.71 184.15 0)
-      (effects (font (size 1.27 1.27)) (justify left) hide)
+    (property "Value" "ERB-RD2R00X " (at 88.265 184.785 90)
+      (effects (font (size 1.27 1.27)) (justify left))
     )
     (property "Footprint" "Fuse:Fuse_0402_1005Metric" (at 89.027 182.88 90)
@@
     )
     (property "Datasheet" "~" (at 90.805 182.88 0)
+      (effects (font (size 1.27 1.27)) hide)
+    )
+    (property "description" "Electric Fuse, Fast Blow, 2A, 32VDC, 35A (IR), Surface Mount" (at 90.805 182.88 90)
       (effects (font (size 1.27 1.27)) hide)
     )
@@
       (effects (font (size 1.27 1.27)) (justify left))
     )
-    (property "Footprint" "Connector_PinHeader_2.00mm:PinHeader_1x08_P2.00mm_Horizontal" (at 101.6 203.835 0)
-      (effects (font (size 1.27 1.27)) hide)
-    )
+    (property "Footprint" "Connector_PinSocket_2.54mm:PinSocket_1x08_P2.54mm_Horizontal" (at 101.6 203.835 0)
+      (effects (font (size 1.27 1.27)) hide)
+    )
