File: Schematic/Kicad_Schematic/Flipper_Zero_DIY/Power_and_Vibro.kicad_sch (KiCad schematic)
At the start: 0 parts

Commit message: finished Su-1-GHz-CC1101
Other:
- company: Flipper Devices Inc. -> Originally from : Flipper Devices Inc.
Changed lines of the file:
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@@
     (title "Flipper Device DIY")
     (rev "13.F7B9C6")
-    (company "Flipper Devices Inc.")
+    (company "Originally from : Flipper Devices Inc.")
+    (comment 1 "DIY Version 1.0")
   )
 )

Commit message: Finished RFID Schematic
Parts:
- added Q1: NMOS, symbol Simulation_SPICE:NMOS
- added RC35: 10uF, symbol Device:C
- added RC36: 22uF, symbol Device:C
- added RDA: FAN48610BUC50X, WLCSP9_1P2X1P2_ONS, symbol FAN48610BUC50X:FAN48610BUC50X
- added RL3: 470nH, symbol Device:L
- added RR3: 22, symbol Device:R
- added RR4: 150, symbol Device:R
- added RR5: 10k, symbol Device:R
- added RVD2: 1N4148X-TP, symbol Device:D
- added RX10: PCB_PAD, symbol Connector:Conn_01x02_Socket
- added RX3: FH34SRJ-18S-0.5SH(50), symbol Connector:Conn_01x18_Socket
- added TP69: IR_RX, symbol Connector:TestPoint
- added TP70: IR_TX, symbol Connector:TestPoint
- added TP71: SPEAKER, symbol Connector:TestPoint
- added TP72: iBTN, symbol Connector:TestPoint
- added TP73: SPI_R_MOSI, symbol Connector:TestPoint
- added TP74: NFC_CS, symbol Connector:TestPoint
- added TP75: VIBRO1, symbol Connector:TestPoint
- added TP76: RFID_OUT, symbol Connector:TestPoint
- added TP77: RFID_PULL, symbol Connector:TestPoint
- added TP78: SPI_R_MISO, symbol Connector:TestPoint
- added TP79: SPI_R_SCK, symbol Connector:TestPoint
- added TP80: RFID_RF_IN, symbol Connector:TestPoint
- added TP81: GND2, symbol Connector:TestPoint
- added TP82: GND3, symbol Connector:TestPoint
- added TP83: RFID_CARRIER, symbol Connector:TestPoint
- added TP84: VIBRO2, symbol Connector:TestPoint
- added TP85: VIBRO3, symbol Connector:TestPoint
- added TP86: SYS1, symbol Connector:TestPoint
- added TP87: SYS2, symbol Connector:TestPoint
- added TP88: 5V_1, symbol Connector:TestPoint
- added TP89: 5V_2, symbol Connector:TestPoint
- added TP90: 3V_1, symbol Connector:TestPoint
- added TP91: 3V_2, symbol Connector:TestPoint
- added TP92: GND_1, symbol Connector:TestPoint
- added TP93: GND_2, symbol Connector:TestPoint
Connections:
- new net: Q1.2 (G), RR4.1, RR5.1
- new net: RR4.2, RX3.10 (Pin_10), TP75.1
- new net: RR3.2, RVD2.1 (K), RX10.1 (Pin_1), TP85.1
- new net: Q1.1 (D), RVD2.2 (A), RX10.2 (Pin_2), TP84.1
- new net: RDA.B1 (SW), RDA.B2 (SW), RL3.2
- new net +3V3: RX3.3 (Pin_3), TP90.1, TP91.1
- new net +5V: RC36.1, RDA.A1 (VOUT), RDA.A2 (VOUT), TP88.1, TP89.1
- new net GNDREF: Q1.3 (S), RC35.2, RC36.2, RDA.C1 (PGND), RDA.C2 (PGND), RDA.C3 (AGND), RR5.2, RX3.6 (Pin_6), RX3.8 (Pin_8), TP81.1, TP82.1, TP92.1, TP93.1
- new net IR_RX: RX3.17 (Pin_17), TP69.1
- new net IR_TX: RX3.16 (Pin_16), TP70.1
- new net NFC_CS: RX3.4 (Pin_4), TP74.1
- new net RFID_CARRIER: RX3.18 (Pin_18), TP83.1
- new net RFID_OUT: RX3.12 (Pin_12), TP76.1
- new net RFID_PULL: RX3.11 (Pin_11), TP77.1
- new net RFID_RF_IN: RX3.5 (Pin_5), TP80.1
- new net SPEAKER: RX3.15 (Pin_15), TP71.1
- new net SPI_R_MISO: RX3.9 (Pin_9), TP78.1
- new net SPI_R_MOSI: RX3.13 (Pin_13), TP73.1
- new net SPI_R_SCK: RX3.7 (Pin_7), TP79.1
- new net SYS: RC35.1, RDA.A3 (VIN), RDA.B3 (EN), RL3.1, RR3.1, RX3.1 (Pin_1), RX3.2 (Pin_2), TP86.1, TP87.1
- new net iBTN: RX3.14 (Pin_14), TP72.1
Other:
- note added: "+3.3V"
- note added: "GND"
- note added: "IR_RX"
- note added: "IR_TX"
- note added: "RFID_CARROER"
- note added: "RFID_IN"
- note added: "RFID_OUT"
- note added: "RFID_PULL"
- note added: "SPEAKER"
- note added: "ST25 BSS"
- note added: "ST25 SCLK"
- note added: "ST25_MISO"
- note added: "ST25_MOSI"
- note added: "SYS"
- note added: "VIBRO"
- note added: "Vibro+"
- note added: "Vibro-"
- note added: "iBTN"
