File: Schematic/Kicad_Schematic/Flipper_Zero_DIY/RFID.kicad_sch (KiCad schematic)
At the start: 0 parts

Commit message: finished Su-1-GHz-CC1101
Other:
- company: Flipper Devices Inc. -> Originally from : Flipper Devices Inc.
Changed lines of the file:
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@@
     (title "Flipper Device DIY")
     (rev "13.F7B9C6")
-    (company "Flipper Devices Inc.")
+    (company "Originally from : Flipper Devices Inc.")
+    (comment 1 "DIY Version 1.0")
   )
 )
